File: eagle/MatrixPi.sch (EAGLE design)
At the start: 0 parts

Commit message: Added WIP eagle board and schematic
Parts:
- added A0, A1, A2: (no value), microbuilder:SOLDERJUMPERREFLOW_NOPASTE
- added C1, C2, C3: 10uF, rcl:C-EUC0805
- added D1: 1N4148, adafruit:DIODESOD-323F
- added LED1, LED2: (no value), matrix_parts:MATRIX_8X8_ROWCATHODE
- added R1, R2, R3, R4, R5: 10K, resistor:R-EU_M0805
- added SV1: (no value), con-lstb:MA05-2
- added SV2: (no value), con-lstb:MA03-1
- added U2: 28-SOIC, microbuilder:HT16K33_SOP28
Connections:
- new net +5V: SV1.2, SV1.4
- new net A0: A0.2, LED1.A3, U2.ROW2/A0
- new net A1: A1.2, LED1.A2, U2.ROW1/A1
- new net A2: A2.2, LED1.A1, U2.ROW0/A2
- new net GND: C1.2, C2.2, C3.2, SV1.6, SV1.9, SV2.2, U2.VSS
- new net GPIO4: SV1.7
- new net N$1: LED1.K8, LED2.K8, U2.COM7
- new net N$10: LED2.A7, U2.ROW14/K12
- new net N$11: LED2.A6, U2.ROW13/K11
- new net N$12: LED2.A8, U2.ROW15/K13/INT
- new net N$16: D1.C, R3.1, R4.1, R5.1
- new net N$19: A1.1, R3.2
- new net N$2: LED1.K7, LED2.K7, U2.COM6
- new net N$20: A0.1, R4.2
- new net N$22: LED1.A8, U2.ROW7/K5
- new net N$23: LED1.A7, U2.ROW6/K4
- new net N$25: LED1.A5, U2.ROW4/K2
- new net N$26: LED1.A4, U2.ROW3/K1
- new net N$3: LED1.K6, LED2.K6, U2.COM5
- new net N$35: LED1.A6, U2.ROW5/K3
- new net N$38: LED2.A1, U2.ROW8/K6
- new net N$39: LED2.A2, U2.ROW9/K7
- new net N$4: LED1.K5, LED2.K5, U2.COM4
- new net N$40: LED2.A4, U2.ROW11/K9
- new net N$41: LED2.A3, U2.ROW10/K8
- new net N$42: LED2.A5, U2.ROW12/K10
- new net N$5: LED1.K4, LED2.K4, U2.COM3/KS2
- new net N$6: LED1.K3, LED2.K3, U2.COM2/KS1
- new net N$7: LED1.K2, LED2.K2, U2.COM1/KS0
- new net N$8: D1.A, LED1.K1, LED2.K1, U2.COM0/AD
- new net N$9: A2.1, R5.2
- new net RXD0: SV1.10
- new net SCL: R1.2, SV1.5, SV2.3, U2.SCL
- new net SDA: R2.2, SV1.3, SV2.1, U2.SDA
- new net TXD0: SV1.8
- new net VDD: C1.1, C2.1, C3.1, R1.1, R2.1, SV1.1, U2.VDD
