File: eagle/MatrixPi.brd (EAGLE design)
At the start: 85 x 56 mm, 17 parts, among them U2 28-SOIC

Commit message: Revised board
Parts:
- moved R1 39.9 mm to (62.9, 23.7), turned to 90 degrees
- moved R2 36.3 mm to (60.9, 23.7), turned to 90 degrees
- moved A0 29.6 mm to (44.0, 15.0)
- moved R4 29.5 mm to (44.0, 11.0)
- moved D1 25.9 mm to (41.5, 10.6)
- moved A1 25.8 mm to (46.0, 15.0)
- moved R3 25.7 mm to (46.0, 11.0)
- moved A2 22.0 mm to (48.0, 15.0)
- moved R5 21.9 mm to (48.0, 11.0)
- moved C1 4.53 mm to (54.1, 23.7), turned to 270 degrees
- moved LED1 4.50 mm to (61.5, 28.0)
- moved LED2 4.50 mm to (23.5, 28.0)
- moved U2 4.27 mm to (42.5, 28.0)
- moved C2 1.95 mm to (56.1, 23.7), turned to 270 degrees
- moved C3 1.70 mm to (58.1, 23.7), turned to 270 degrees
Routing:
- net SCL: track 0.00 -> 18.1 mm
- net SDA: track 0.00 -> 14.5 mm
- net VDD: track 13.6 -> 15.8 mm

Commit message: Revised board
Parts:
- moved R1 41.2 mm to (22.6, 32.2), turned to 270 degrees
- moved R2 37.2 mm to (24.7, 32.2), turned to 270 degrees
- moved D1 32.8 mm to (47.8, 42.8), turned to 180 degrees
- moved R5 32.1 mm to (39.1, 41.8), turned to 270 degrees
- moved C3 31.8 mm to (27.4, 32.2), turned to 90 degrees
- moved R3 31.2 mm to (41.1, 41.8), turned to 270 degrees
- moved R4 30.8 mm to (43.1, 41.8), turned to 270 degrees
- moved C2 28.0 mm to (29.5, 32.2), turned to 90 degrees
- moved A2 24.5 mm to (39.1, 37.8), turned to 270 degrees
- moved C1 24.3 mm to (31.4, 32.2), turned to 90 degrees
- moved A1 23.3 mm to (41.1, 37.8), turned to 270 degrees
- moved A0 22.8 mm to (43.1, 37.8), turned to 270 degrees
- turned U2 to 0 degrees
Routing:
- net SCL: track 18.1 -> 61.0 mm
- net SDA: track 14.5 -> 54.2 mm
- net VDD: track 15.8 -> 37.2 mm, vias 0 -> 2
- net N$16: track 0.00 -> 7.74 mm
- net A0: track 0.00 -> 5.32 mm
- net A1: track 0.00 -> 4.73 mm
- net A2: track 0.00 -> 4.39 mm
- net N$8: track 0.00 -> 4.12 mm
- net N$9: track 0.00 -> 2.29 mm
- net N$20: track 0.00 -> 2.29 mm
- net N$19: track 0.00 -> 2.29 mm
Other:
- board text removed: "A0"
- board text removed: "A1"
- board text removed: "A2"

Commit message: Board revisions
Parts:
- moved R1 39.5 mm to (62.1, 32.2), flipped to the bottom
- moved R2 35.4 mm to (60.1, 32.2), flipped to the bottom
- moved C3 29.8 mm to (57.2, 32.2), flipped to the bottom
- moved C2 25.7 mm to (55.1, 32.2), flipped to the bottom
- moved C1 21.7 mm to (53.1, 32.2), flipped to the bottom
- moved D1 14.8 mm to (33.4, 45.9), flipped to the bottom
- moved A2 7.61 mm to (46.0, 41.0), flipped to the bottom
- moved R5 7.61 mm to (46.0, 45.0), flipped to the bottom
- moved A1 4.00 mm to (43.5, 41.0), flipped to the bottom
- moved R3 4.00 mm to (43.5, 45.0), flipped to the bottom
- moved A0 3.83 mm to (41.0, 41.0), flipped to the bottom
- moved R4 3.83 mm to (41.0, 45.0), flipped to the bottom
- flipped LED1 to the top
- flipped LED2 to the top
- turned SV2 to 270 degrees
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Routing:
- net N$23: track 0.00 -> 23.7 mm, vias 0 -> 2
- net A2: track 4.39 -> 27.1 mm, vias 0 -> 2
- net N$22: track 0.00 -> 22.5 mm, vias 0 -> 2
- net VDD: track 37.2 -> 55.8 mm, vias 2 -> 1
- net SDA: track 54.2 -> 69.3 mm, vias 0 -> 1
- net SCL: track 61.0 -> 69.0 mm, vias 0 -> 1
- net N$16: track 7.74 -> 11.7 mm
- net A1: track 4.73 -> 8.06 mm
- net A0: track 5.32 -> 8.57 mm
- net +5V: track 0.00 -> 2.54 mm

Commit message: Board revision
Routing:
- net N$38: track 0.00 -> 26.5 mm
Changed lines of the file:
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@@
 <contactref element="U2" pad="P$17"/>
 <contactref element="LED2" pad="13"/>
-<wire x1="22.23" y1="41.97" x2="36.785" y2="33.08" width="0" layer="19" extent="16-16"/>
+<wire x1="36.785" y1="33.08" x2="36.785" y2="35.315" width="0.3048" layer="16"/>
+<wire x1="36.785" y1="35.315" x2="31.1" y2="40.95" width="0.3048" layer="16"/>
+<wire x1="31.1" y1="40.95" x2="31.1" y2="43.5" width="0.3048" layer="16"/>
+<wire x1="31.1" y1="43.5" x2="28.2" y2="46.45" width="0.3048" layer="16"/>
+<wire x1="28.2" y1="46.45" x2="23.75" y2="46.45" width="0.3048" layer="16"/>
+<wire x1="23.75" y1="46.45" x2="22.25" y2="44.95" width="0.3048" layer="16"/>
+<wire x1="22.25" y1="44.95" x2="22.25" y2="41.99" width="0.3048" layer="16"/>
+<wire x1="22.25" y1="41.99" x2="22.23" y2="41.97" width="0.3048" layer="16"/>
 </signal>
 <signal name="N$39">

Commit message: Board revision
Routing:
- net N$7: track 0.00 -> 94.2 mm, vias 0 -> 3
- net N$8: track 3.96 -> 37.7 mm
- net N$26: track 0.00 -> 31.5 mm, vias 0 -> 2
- net N$35: track 0.00 -> 30.8 mm, vias 0 -> 2
Changed lines of the file:
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@@
 <contactref element="LED1" pad="14"/>
 <contactref element="LED2" pad="14"/>
-<wire x1="48.215" y1="22.92" x2="57.69" y2="41.97" width="0" layer="19" extent="16-16"/>
-<wire x1="19.69" y1="41.97" x2="48.215" y2="22.92" width="0" layer="19" extent="16-16"/>
+<wire x1="19.69" y1="41.97" x2="19.69" y2="40.01" width="0.3048" layer="16"/>
+<wire x1="19.69" y1="40.01" x2="19.75" y2="39.95" width="0.3048" layer="16"/>
+<via x="19.75" y="39.95" extent="1-16" drill="0.6" shape="octagon"/>
+<wire x1="19.75" y1="39.95" x2="19.75" y2="36.4" width="0.3048" layer="1"/>
+<wire x1="19.75" y1="36.4" x2="31.35" y2="24.8" width="0.3048" layer="1"/>
+<wire x1="31.35" y1="24.8" x2="48.25" y2="24.8" width="0.3048" layer="1"/>
+<wire x1="48.25" y1="24.8" x2="48.3" y2="24.75" width="0.3048" layer="1"/>
+<wire x1="48.3" y1="24.75" x2="48.3" y2="20.85" width="0.3048" layer="1"/>
+<wire x1="48.3" y1="20.85" x2="48.2" y2="20.75" width="0.3048" layer="1"/>
+<via x="48.2" y="20.75" extent="1-16" drill="0.6" shape="octagon"/>
+<wire x1="48.2" y1="20.75" x2="48.2" y2="22.905" width="0.3048" layer="16"/>
+<wire x1="48.2" y1="22.905" x2="48.215" y2="22.92" width="0.3048" layer="16"/>
+<wire x1="57.69" y1="41.97" x2="57.69" y2="40.54" width="0.3048" layer="16"/>
+<wire x1="57.69" y1="40.54" x2="56.65" y2="39.5" width="0.3048" layer="16"/>
+<via x="56.65" y="39.5" extent="1-16" drill="0.6" shape="octagon"/>
+<wire x1="56.65" y1="39.5" x2="57.1" y2="39.5" width="0.3048" layer="1"/>
+<wire x1="57.1" y1="39.5" x2="59" y2="41.4" width="0.3048" layer="1"/>
+<wire x1="59" y1="41.4" x2="59" y2="42.7" width="0.3048" layer="1"/>
+<wire x1="59" y1="42.7" x2="60" y2="43.7" width="0.3048" layer="1"/>
+<wire x1="60" y1="43.7" x2="68.35" y2="43.7" width="0.3048" layer="1"/>
+<wire x1="68.35" y1="43.7" x2="69.2" y2="42.85" width="0.3048" layer="1"/>
+<wire x1="69.2" y1="42.85" x2="69.2" y2="39.65" width="0.3048" layer="1"/>
+<wire x1="69.2" y1="39.65" x2="68" y2="38.45" width="0.3048" layer="1"/>
+<wire x1="68" y1="38.45" x2="61.25" y2="38.45" width="0.3048" layer="1"/>
+<wire x1="61.25" y1="38.45" x2="56.15" y2="33.35" width="0.3048" layer="1"/>
+<wire x1="56.15" y1="33.35" x2="56.15" y2="32.7" width="0.3048" layer="1"/>
+<wire x1="56.15" y1="32.7" x2="48.25" y2="24.8" width="0.3048" layer="1"/>
 </signal>
 <signal name="N$8">
@@
 <wire x1="32.377" y1="45.922" x2="32.377" y2="41.983" width="0.6096" layer="16"/>
 <wire x1="32.377" y1="41.983" x2="32.39" y2="41.97" width="0.6096" layer="16"/>
-<wire x1="49.485" y1="22.92" x2="70.39" y2="41.97" width="0" layer="19" extent="16-16"/>
-<wire x1="32.39" y1="41.97" x2="49.485" y2="22.92" width="0" layer="19" extent="16-16"/>
+<wire x1="70.39" y1="41.97" x2="70.39" y2="35.04" width="0.3048" layer="16"/>
+<wire x1="70.39" y1="35.04" x2="63.25" y2="27.9" width="0.3048" layer="16"/>
+<wire x1="63.25" y1="27.9" x2="52.95" y2="27.9" width="0.3048" layer="16"/>
+<wire x1="52.95" y1="27.9" x2="49.5" y2="24.45" width="0.3048" layer="16"/>
+<wire x1="49.5" y1="24.45" x2="49.5" y2="22.935" width="0.3048" layer="16"/>
+<wire x1="49.5" y1="22.935" x2="49.485" y2="22.92" width="0.3048" layer="16"/>
+<wire x1="49.5" y1="24.45" x2="32.39" y2="41.97" width="0" layer="19" extent="16-16"/>
 </signal>
 <signal name="VDD">
@@
 <contactref element="U2" pad="P$22"/>
 <contactref element="LED1" pad="10"/>
-<wire x1="43.135" y1="33.08" x2="67.85" y2="41.97" width="0" layer="19" extent="16-16"/>
+<wire x1="43.135" y1="33.08" x2="43.135" y2="35.235" width="0.3048" layer="16"/>
+<wire x1="43.135" y1="35.235" x2="43.15" y2="35.25" width="0.3048" layer="16"/>
+<via x="43.15" y="35.25" extent="1-16" drill="0.6" shape="octagon"/>
+<wire x1="43.15" y1="35.25" x2="44.8" y2="35.25" width="0.3048" layer="1"/>
+<wire x1="44.8" y1="35.25" x2="45.95" y2="34.35" width="0.3048" layer="1"/>
+<wire x1="45.95" y1="34.35" x2="55.25" y2="34.35" width="0.3048" layer="1"/>
+<wire x1="55.25" y1="34.35" x2="60.55" y2="39.65" width="0.3048" layer="1"/>
+<wire x1="60.55" y1="39.65" x2="67.35" y2="39.65" width="0.3048" layer="1"/>
+<wire x1="67.35" y1="39.65" x2="67.9" y2="40.2" width="0.3048" layer="1"/>
+<via x="67.9" y="40.2" extent="1-16" drill="0.6" shape="octagon"/>
+<wire x1="67.9" y1="40.2" x2="67.9" y2="41.92" width="0.3048" layer="16"/>
+<wire x1="67.9" y1="41.92" x2="67.85" y2="41.97" width="0.3048" layer="16"/>
 </signal>
 <signal name="N$35">
 <contactref element="U2" pad="P$20"/>
 <contactref element="LED1" pad="11"/>
-<wire x1="40.595" y1="33.08" x2="65.31" y2="41.97" width="0" layer="19" extent="16-16"/>
+<wire x1="40.595" y1="33.08" x2="40.595" y2="35.545" width="0.3048" layer="16"/>
+<wire x1="40.595" y1="35.545" x2="41.35" y2="36.3" width="0.3048" layer="16"/>
+<via x="41.35" y="36.3" extent="1-16" drill="0.6" shape="octagon"/>
+<wire x1="41.35" y1="36.3" x2="45.25" y2="36.3" width="0.3048" layer="1"/>
+<wire x1="45.25" y1="36.3" x2="46.35" y2="35.2" width="0.3048" layer="1"/>
+<wire x1="46.35" y1="35.2" x2="54.35" y2="35.2" width="0.3048" layer="1"/>
+<wire x1="54.35" y1="35.2" x2="59.85" y2="40.7" width="0.3048" layer="1"/>
+<wire x1="59.85" y1="40.7" x2="64.2" y2="40.7" width="0.3048" layer="1"/>
+<wire x1="64.2" y1="40.7" x2="64.25" y2="40.75" width="0.3048" layer="1"/>
+<via x="64.25" y="40.75" extent="1-16" drill="0.6" shape="octagon"/>
+<wire x1="64.25" y1="40.75" x2="64.25" y2="40.91" width="0.3048" layer="16"/>
+<wire x1="64.25" y1="40.91" x2="65.31" y2="41.97" width="0.3048" layer="16"/>
 </signal>
 <signal name="N$38">

Commit message: Board revision
Routing:
- net N$3: track 0.00 -> 67.3 mm, vias 0 -> 2
- net N$6: track 0.00 -> 60.6 mm
- net N$1: track 0.00 -> 57.5 mm, vias 0 -> 4
- net N$5: track 0.00 -> 38.7 mm
- net N$8: track 37.7 -> 39.9 mm
Changed lines of the file:
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@@
 <contactref element="LED1" pad="5"/>
 <contactref element="LED2" pad="5"/>
-<wire x1="40.595" y1="22.92" x2="62.77" y2="14.03" width="0" layer="19" extent="16-16"/>
-<wire x1="24.77" y1="14.03" x2="40.595" y2="22.92" width="0" layer="19" extent="16-16"/>
+<wire x1="62.77" y1="14.03" x2="62.77" y2="10.72" width="0.3048" layer="16"/>
+<wire x1="62.77" y1="10.72" x2="61.5" y2="9.45" width="0.3048" layer="16"/>
+<wire x1="61.5" y1="9.45" x2="48.3" y2="9.45" width="0.3048" layer="16"/>
+<wire x1="48.3" y1="9.45" x2="48.2" y2="9.75" width="0.3048" layer="16"/>
+<via x="48.2" y="9.75" extent="1-16" drill="0.6" shape="octagon"/>
+<wire x1="48.2" y1="9.75" x2="44.9" y2="9.8" width="0.3048" layer="1"/>
+<via x="44.9" y="9.8" extent="1-16" drill="0.6" shape="octagon"/>
+<wire x1="44.9" y1="9.8" x2="40.5" y2="9.55" width="0.3048" layer="16"/>
+<wire x1="40.5" y1="9.55" x2="37.25" y2="9.55" width="0.3048" layer="16"/>
+<wire x1="37.25" y1="9.55" x2="37.2" y2="9.7" width="0.3048" layer="16"/>
+<via x="37.2" y="9.7" extent="1-16" drill="0.6" shape="octagon"/>
+<wire x1="37.2" y1="9.7" x2="31.55" y2="9.5" width="0.3048" layer="1"/>
+<wire x1="31.55" y1="9.5" x2="31.45" y2="9.4" width="0.3048" layer="1"/>
+<via x="31.45" y="9.4" extent="1-16" drill="0.6" shape="octagon"/>
+<wire x1="31.45" y1="9.4" x2="29.4" y2="9.4" width="0.3048" layer="16"/>
+<wire x1="29.4" y1="9.4" x2="24.77" y2="14.03" width="0.3048" layer="16"/>
+<wire x1="40.595" y1="22.92" x2="40.595" y2="9.645" width="0.3048" layer="16"/>
+<wire x1="40.595" y1="9.645" x2="40.5" y2="9.55" width="0.3048" layer="16"/>
 </signal>
 <signal name="N$2">
@@
 <contactref element="LED1" pad="7"/>
 <contactref element="LED2" pad="7"/>
-<wire x1="43.135" y1="22.92" x2="67.85" y2="14.03" width="0" layer="19" extent="16-16"/>
-<wire x1="29.85" y1="14.03" x2="43.135" y2="22.92" width="0" layer="19" extent="16-16"/>
+<wire x1="67.85" y1="14.03" x2="67.85" y2="10.55" width="0.3048" layer="16"/>
+<wire x1="67.85" y1="10.55" x2="64.65" y2="7.35" width="0.3048" layer="16"/>
+<wire x1="64.65" y1="7.35" x2="35.2" y2="7.35" width="0.3048" layer="16"/>
+<wire x1="35.2" y1="7.35" x2="30.95" y2="11.6" width="0.3048" layer="16"/>
+<wire x1="30.95" y1="11.6" x2="30.95" y2="12.93" width="0.3048" layer="16"/>
+<wire x1="30.95" y1="12.93" x2="29.85" y2="14.03" width="0.3048" layer="16"/>
+<wire x1="30.95" y1="12.93" x2="30.95" y2="14.45" width="0.3048" layer="16"/>
+<wire x1="30.95" y1="14.45" x2="32.05" y2="15.55" width="0.3048" layer="16"/>
+<wire x1="32.05" y1="15.55" x2="39.2" y2="15.55" width="0.3048" layer="16"/>
+<wire x1="39.2" y1="15.55" x2="39.25" y2="15.6" width="0.3048" layer="16"/>
+<via x="39.25" y="15.6" extent="1-16" drill="0.6" shape="octagon"/>
+<wire x1="39.25" y1="15.6" x2="42.2" y2="15.6" width="0.3048" layer="1"/>
+<via x="42.2" y="15.6" extent="1-16" drill="0.6" shape="octagon"/>
+<wire x1="42.2" y1="15.6" x2="43.135" y2="16.535" width="0.3048" layer="16"/>
+<wire x1="43.135" y1="16.535" x2="43.135" y2="22.92" width="0.3048" layer="16"/>
 </signal>
 <signal name="N$4">
@@
 <contactref element="LED1" pad="8"/>
 <contactref element="LED2" pad="8"/>
-<wire x1="46.945" y1="22.92" x2="70.39" y2="14.03" width="0" layer="19" extent="16-16"/>
-<wire x1="32.39" y1="14.03" x2="46.945" y2="22.92" width="0" layer="19" extent="16-16"/>
+<wire x1="70.39" y1="14.03" x2="70.22" y2="14.03" width="0.3048" layer="16"/>
+<wire x1="70.22" y1="14.03" x2="68.85" y2="15.4" width="0.3048" layer="16"/>
+<wire x1="68.85" y1="15.4" x2="67.45" y2="15.4" width="0.3048" layer="16"/>
+<wire x1="67.45" y1="15.4" x2="66.6" y2="14.55" width="0.3048" layer="16"/>
+<wire x1="66.6" y1="14.55" x2="66.6" y2="11.55" width="0.3048" layer="16"/>
+<wire x1="66.6" y1="11.55" x2="63.75" y2="8.7" width="0.3048" layer="16"/>
+<wire x1="63.75" y1="8.7" x2="46.85" y2="8.7" width="0.3048" layer="16"/>
+<wire x1="46.85" y1="8.7" x2="36.1" y2="8.7" width="0.3048" layer="16"/>
+<wire x1="36.1" y1="8.7" x2="32.25" y2="12.55" width="0.3048" layer="16"/>
+<wire x1="32.25" y1="12.55" x2="32.25" y2="13.89" width="0.3048" layer="16"/>
+<wire x1="32.25" y1="13.89" x2="32.39" y2="14.03" width="0.3048" layer="16"/>
+<wire x1="46.945" y1="22.92" x2="46.945" y2="8.795" width="0.3048" layer="16"/>
+<wire x1="46.945" y1="8.795" x2="46.85" y2="8.7" width="0.3048" layer="16"/>
 </signal>
 <signal name="N$7">
@@
 <wire x1="59" y1="42.7" x2="60" y2="43.7" width="0.3048" layer="1"/>
 <wire x1="60" y1="43.7" x2="68.35" y2="43.7" width="0.3048" layer="1"/>
-<wire x1="68.35" y1="43.7" x2="69.2" y2="42.85" width="0.3048" layer="1"/>
-<wire x1="69.2" y1="42.85" x2="69.2" y2="39.65" width="0.3048" layer="1"/>
-<wire x1="69.2" y1="39.65" x2="68" y2="38.45" width="0.3048" layer="1"/>
+<wire x1="68.35" y1="43.7" x2="69.1" y2="42.85" width="0.3048" layer="1"/>
+<wire x1="69.1" y1="42.85" x2="69.1" y2="39.65" width="0.3048" layer="1"/>
+<wire x1="69.1" y1="39.65" x2="68" y2="38.45" width="0.3048" layer="1"/>
 <wire x1="68" y1="38.45" x2="61.25" y2="38.45" width="0.3048" layer="1"/>
 <wire x1="61.25" y1="38.45" x2="56.15" y2="33.35" width="0.3048" layer="1"/>
@@
 <wire x1="32.377" y1="45.922" x2="32.377" y2="41.983" width="0.6096" layer="16"/>
 <wire x1="32.377" y1="41.983" x2="32.39" y2="41.97" width="0.6096" layer="16"/>
-<wire x1="70.39" y1="41.97" x2="70.39" y2="35.04" width="0.3048" layer="16"/>
-<wire x1="70.39" y1="35.04" x2="63.25" y2="27.9" width="0.3048" layer="16"/>
-<wire x1="63.25" y1="27.9" x2="52.95" y2="27.9" width="0.3048" layer="16"/>
-<wire x1="52.95" y1="27.9" x2="49.5" y2="24.45" width="0.3048" layer="16"/>
-<wire x1="49.5" y1="24.45" x2="49.5" y2="22.935" width="0.3048" layer="16"/>
+<wire x1="70.39" y1="41.97" x2="70.39" y2="31.04" width="0.3048" layer="16"/>
+<wire x1="70.39" y1="31.04" x2="64.5" y2="25.15" width="0.3048" layer="16"/>
+<wire x1="64.5" y1="25.15" x2="50.5" y2="25.15" width="0.3048" layer="16"/>
+<wire x1="50.5" y1="25.15" x2="49.5" y2="24.15" width="0.3048" layer="16"/>
+<wire x1="49.5" y1="24.15" x2="49.5" y2="22.935" width="0.3048" layer="16"/>
 <wire x1="49.5" y1="22.935" x2="49.485" y2="22.92" width="0.3048" layer="16"/>
-<wire x1="49.5" y1="24.45" x2="32.39" y2="41.97" width="0" layer="19" extent="16-16"/>
+<wire x1="50.5" y1="25.15" x2="32.39" y2="41.97" width="0" layer="19" extent="16-16"/>
 </signal>
 <signal name="VDD">
@@
 <contactref element="LED1" pad="12"/>
 <contactref element="LED2" pad="12"/>
-<wire x1="45.675" y1="22.92" x2="62.77" y2="41.97" width="0" layer="19" extent="16-16"/>
-<wire x1="24.77" y1="41.97" x2="45.675" y2="22.92" width="0" layer="19" extent="16-16"/>
+<wire x1="62.77" y1="41.97" x2="62.77" y2="37.88" width="0.3048" layer="16"/>
+<wire x1="62.77" y1="37.88" x2="66.5" y2="34.15" width="0.3048" layer="16"/>
+<wire x1="66.5" y1="34.15" x2="66.5" y2="29.05" width="0.3048" layer="16"/>
+<wire x1="66.5" y1="29.05" x2="63.75" y2="26.3" width="0.3048" layer="16"/>
+<wire x1="63.75" y1="26.3" x2="47.65" y2="26.3" width="0.3048" layer="16"/>
+<wire x1="47.65" y1="26.3" x2="45.65" y2="24.3" width="0.3048" layer="16"/>
+<wire x1="45.65" y1="24.3" x2="45.65" y2="22.945" width="0.3048" layer="16"/>
+<wire x1="45.65" y1="22.945" x2="45.675" y2="22.92" width="0.3048" layer="16"/>
+<wire x1="24.77" y1="41.97" x2="45.65" y2="24.3" width="0" layer="19" extent="16-16"/>
 </signal>
 <signal name="+5V">

Commit message: Eagle files revision number big
Routing:
- net N$7: track 94.0 -> 0.00 mm, vias 3 -> 0
- net N$3: track 67.3 -> 0.00 mm, vias 2 -> 0
- net N$6: track 60.6 -> 0.00 mm
- net N$1: track 57.5 -> 0.00 mm, vias 4 -> 0
- net N$35: track 30.8 -> 33.9 mm
- net A2: track 27.1 -> 24.6 mm
- net N$23: track 23.7 -> 21.6 mm
- net N$22: track 22.5 -> 20.6 mm
- net N$26: track 31.5 -> 30.5 mm

Commit message: Board revision big+1
Routing:
- net N$6: track 0.00 -> 80.3 mm, vias 0 -> 2
- net N$3: track 0.00 -> 78.4 mm, vias 0 -> 2
- net N$4: track 0.00 -> 61.3 mm, vias 0 -> 2
- net N$5: track 38.7 -> 77.2 mm, vias 0 -> 2
- net N$7: track 0.00 -> 34.6 mm, vias 0 -> 2
- net N$8: track 39.9 -> 72.8 mm, vias 0 -> 2
- net N$42: track 0.00 -> 14.1 mm
- net N$22: track 20.6 -> 22.8 mm
- net N$23: track 21.6 -> 23.0 mm
- net N$35: track 33.9 -> 34.5 mm
