File: eagle/MatrixPi.brd (EAGLE design)
At the start: 85 x 56 mm, 17 parts, among them U2 28-SOIC

Commit message: Board revision big+2
Routing:
- net N$2: track 0.00 -> 95.1 mm, vias 0 -> 2
Changed lines of the file:
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@@
 <contactref element="LED1" pad="2"/>
 <contactref element="LED2" pad="2"/>
-<wire x1="41.865" y1="22.92" x2="55.15" y2="14.03" width="0" layer="19" extent="16-16"/>
-<wire x1="17.15" y1="14.03" x2="41.865" y2="22.92" width="0" layer="19" extent="16-16"/>
+<wire x1="17.15" y1="14.03" x2="17.15" y2="12.25" width="0.4064" layer="16"/>
+<via x="17.15" y="12.25" extent="1-16" drill="0.6" shape="octagon"/>
+<wire x1="17.15" y1="12.25" x2="21.4" y2="8" width="0.4064" layer="1"/>
+<wire x1="21.4" y1="8" x2="26.55" y2="8" width="0.4064" layer="1"/>
+<wire x1="26.55" y1="8" x2="28.25" y2="6.3" width="0.4064" layer="1"/>
+<wire x1="28.25" y1="6.3" x2="28.25" y2="2.65" width="0.4064" layer="1"/>
+<wire x1="28.25" y1="2.65" x2="28.65" y2="2.25" width="0.4064" layer="1"/>
+<wire x1="28.65" y1="2.25" x2="30.15" y2="2.25" width="0.4064" layer="1"/>
+<wire x1="30.15" y1="2.25" x2="33.9" y2="6" width="0.4064" layer="1"/>
+<wire x1="33.9" y1="6" x2="34.15" y2="6" width="0.4064" layer="1"/>
+<via x="34.15" y="6" extent="1-16" drill="0.6" shape="octagon"/>
+<wire x1="34.15" y1="6" x2="36.85" y2="3.3" width="0.4064" layer="16"/>
+<wire x1="36.85" y1="3.3" x2="54.35" y2="3.3" width="0.4064" layer="16"/>
+<wire x1="54.35" y1="3.3" x2="55.15" y2="4.1" width="0.4064" layer="16"/>
+<wire x1="55.15" y1="4.1" x2="55.15" y2="14.03" width="0.4064" layer="16"/>
+<wire x1="41.865" y1="22.92" x2="41.865" y2="25.735" width="0.4064" layer="16"/>
+<wire x1="41.865" y1="25.735" x2="41.3" y2="26.3" width="0.4064" layer="16"/>
+<wire x1="41.3" y1="26.3" x2="23.8" y2="26.3" width="0.4064" layer="16"/>
+<wire x1="23.8" y1="26.3" x2="17.2" y2="19.7" width="0.4064" layer="16"/>
+<wire x1="17.2" y1="19.7" x2="17.2" y2="14.08" width="0.4064" layer="16"/>
+<wire x1="17.2" y1="14.08" x2="17.15" y2="14.03" width="0.4064" layer="16"/>
 </signal>
 <signal name="N$3">

Commit message: Board revision big+3
Routing:
- net N$1: track 0.00 -> 70.7 mm, vias 0 -> 5

Commit message: Board revision big+4
Routing:
- net N$39: track 0.00 -> 102.7 mm
- net N$41: track 0.00 -> 86.7 mm
- net N$12: track 0.00 -> 60.7 mm, vias 0 -> 2
- net N$10: track 0.00 -> 50.4 mm, vias 0 -> 2
- net N$11: track 0.00 -> 26.4 mm, vias 0 -> 2
- net N$40: track 0.00 -> 21.9 mm, vias 0 -> 2
Changed lines of the file:
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@@
 <contactref element="U2" pad="P$11"/>
 <contactref element="LED2" pad="15"/>
-<wire x1="17.15" y1="41.97" x2="38.055" y2="22.92" width="0" layer="19" extent="16-16"/>
+<wire x1="38.055" y1="22.92" x2="38.05" y2="22.915" width="0.3048" layer="16"/>
+<wire x1="38.05" y1="22.915" x2="38.05" y2="19.65" width="0.3048" layer="16"/>
+<via x="38.05" y="19.65" extent="1-16" drill="0.6" shape="octagon"/>
+<wire x1="38.05" y1="19.65" x2="37.05" y2="18.65" width="0.3048" layer="1"/>
+<wire x1="37.05" y1="18.65" x2="25.9" y2="18.65" width="0.3048" layer="1"/>
+<wire x1="25.9" y1="18.65" x2="22.95" y2="15.7" width="0.3048" layer="1"/>
+<wire x1="22.95" y1="15.7" x2="20.05" y2="15.7" width="0.3048" layer="1"/>
+<wire x1="20.05" y1="15.7" x2="19.4" y2="16.35" width="0.3048" layer="1"/>
+<wire x1="19.4" y1="16.35" x2="19.4" y2="21.1" width="0.3048" layer="1"/>
+<wire x1="19.4" y1="21.1" x2="18.85" y2="21.65" width="0.3048" layer="1"/>
+<wire x1="18.85" y1="21.65" x2="18.85" y2="23.9" width="0.3048" layer="1"/>
+<via x="18.85" y="23.9" extent="1-16" drill="0.6" shape="octagon"/>
+<wire x1="18.85" y1="23.9" x2="17.15" y2="25.6" width="0.3048" layer="16"/>
+<wire x1="17.15" y1="25.6" x2="17.15" y2="41.97" width="0.3048" layer="16"/>
 </signal>
 <signal name="N$11">
 <contactref element="U2" pad="P$12"/>
 <contactref element="LED2" pad="11"/>
-<wire x1="36.785" y1="22.92" x2="27.31" y2="41.97" width="0" layer="19" extent="16-16"/>
+<wire x1="36.785" y1="22.92" x2="36.785" y2="25.25" width="0.3048" layer="16"/>
+<wire x1="36.785" y1="25.25" x2="31" y2="25.25" width="0.3048" layer="16"/>
+<via x="31" y="25.25" extent="1-16" drill="0.6" shape="octagon"/>
+<wire x1="31" y1="25.25" x2="31" y2="35.55" width="0.3048" layer="1"/>
+<wire x1="31" y1="35.55" x2="27.35" y2="39.2" width="0.3048" layer="1"/>
+<via x="27.35" y="39.2" extent="1-16" drill="0.6" shape="octagon"/>
+<wire x1="27.35" y1="39.2" x2="27.35" y2="41.93" width="0.3048" layer="16"/>
+<wire x1="27.35" y1="41.93" x2="27.31" y2="41.97" width="0.3048" layer="16"/>
 </signal>
 <signal name="N$22">
@@
 <contactref element="U2" pad="P$16"/>
 <contactref element="LED2" pad="3"/>
-<wire x1="19.69" y1="14.03" x2="35.515" y2="33.08" width="0" layer="19" extent="16-16"/>
+<wire x1="35.515" y1="33.08" x2="35.515" y2="35.135" width="0.3048" layer="16"/>
+<wire x1="35.515" y1="35.135" x2="32.45" y2="38" width="0.3048" layer="16"/>
+<wire x1="32.45" y1="38" x2="23.85" y2="38" width="0.3048" layer="16"/>
+<wire x1="23.85" y1="38" x2="20.95" y2="41.1" width="0.3048" layer="16"/>
+<wire x1="20.95" y1="41.1" x2="20.95" y2="43.95" width="0.3048" layer="16"/>
+<wire x1="20.95" y1="43.95" x2="18.5" y2="46.4" width="0.3048" layer="16"/>
+<wire x1="18.5" y1="46.4" x2="8.25" y2="46.4" width="0.3048" layer="16"/>
+<wire x1="8.25" y1="46.4" x2="5.85" y2="44" width="0.3048" layer="16"/>
+<wire x1="5.85" y1="44" x2="5.85" y2="12" width="0.3048" layer="16"/>
+<wire x1="5.85" y1="12" x2="11.3" y2="6.55" width="0.3048" layer="16"/>
+<wire x1="11.3" y1="6.55" x2="17.55" y2="6.55" width="0.3048" layer="16"/>
+<wire x1="17.55" y1="6.55" x2="23.5" y2="12.6" width="0.3048" layer="16"/>
+<wire x1="23.5" y1="12.6" x2="23.5" y2="15.55" width="0.3048" layer="16"/>
+<wire x1="23.5" y1="15.55" x2="22.75" y2="16.4" width="0.3048" layer="16"/>
+<wire x1="22.75" y1="16.4" x2="20.25" y2="16.4" width="0.3048" layer="16"/>
+<wire x1="20.25" y1="16.4" x2="19.7" y2="15.85" width="0.3048" layer="16"/>
+<wire x1="19.7" y1="15.85" x2="19.7" y2="14.04" width="0.3048" layer="16"/>
+<wire x1="19.7" y1="14.04" x2="19.69" y2="14.03" width="0.3048" layer="16"/>
 </signal>
 <signal name="N$40">
 <contactref element="U2" pad="P$14"/>
 <contactref element="LED2" pad="10"/>
-<wire x1="34.245" y1="22.92" x2="29.85" y2="41.97" width="0" layer="19" extent="16-16"/>
+<wire x1="29.85" y1="41.97" x2="30.3" y2="41.52" width="0.3048" layer="16"/>
+<wire x1="30.3" y1="41.52" x2="30.3" y2="39" width="0.3048" layer="16"/>
+<via x="30.3" y="39" extent="1-16" drill="0.6" shape="octagon"/>
+<wire x1="30.3" y1="39" x2="32.45" y2="36.85" width="0.3048" layer="1"/>
+<wire x1="32.45" y1="36.85" x2="32.45" y2="23" width="0.3048" layer="1"/>
+<via x="32.45" y="23" extent="1-16" drill="0.6" shape="octagon"/>
+<wire x1="32.45" y1="23" x2="32.53" y2="22.92" width="0.3048" layer="16"/>
+<wire x1="32.53" y1="22.92" x2="34.245" y2="22.92" width="0.3048" layer="16"/>
 </signal>
 <signal name="N$41">
 <contactref element="U2" pad="P$15"/>
 <contactref element="LED2" pad="4"/>
-<wire x1="22.23" y1="14.03" x2="34.245" y2="33.08" width="0" layer="19" extent="16-16"/>
+<wire x1="34.245" y1="33.08" x2="34.245" y2="35.055" width="0.3048" layer="16"/>
+<wire x1="34.245" y1="35.055" x2="32.45" y2="36.85" width="0.3048" layer="16"/>
+<wire x1="32.45" y1="36.85" x2="21.75" y2="36.85" width="0.3048" layer="16"/>
+<wire x1="21.75" y1="36.85" x2="18.4" y2="40.2" width="0.3048" layer="16"/>
+<wire x1="18.4" y1="40.2" x2="18.4" y2="44.05" width="0.3048" layer="16"/>
+<wire x1="18.4" y1="44.05" x2="17.15" y2="45.3" width="0.3048" layer="16"/>
+<wire x1="17.15" y1="45.3" x2="9.65" y2="45.3" width="0.3048" layer="16"/>
+<wire x1="9.65" y1="45.3" x2="7.65" y2="43.3" width="0.3048" layer="16"/>
+<wire x1="7.65" y1="43.3" x2="7.65" y2="12.15" width="0.3048" layer="16"/>
+<wire x1="7.65" y1="12.15" x2="12.05" y2="7.75" width="0.3048" layer="16"/>
+<wire x1="12.05" y1="7.75" x2="17.05" y2="7.75" width="0.3048" layer="16"/>
+<wire x1="17.05" y1="7.75" x2="22.25" y2="12.95" width="0.3048" layer="16"/>
+<wire x1="22.25" y1="12.95" x2="22.25" y2="14.01" width="0.3048" layer="16"/>
+<wire x1="22.25" y1="14.01" x2="22.23" y2="14.03" width="0.3048" layer="16"/>
 </signal>
 <signal name="N$42">
@@
 <contactref element="U2" pad="P$10"/>
 <contactref element="LED2" pad="16"/>
-<wire x1="14.61" y1="41.97" x2="39.325" y2="22.92" width="0" layer="19" extent="16-16"/>
+<wire x1="39.325" y1="22.92" x2="39.325" y2="19.075" width="0.3048" layer="16"/>
+<wire x1="39.325" y1="19.075" x2="38" y2="17.75" width="0.3048" layer="16"/>
+<via x="38" y="17.75" extent="1-16" drill="0.6" shape="octagon"/>
+<wire x1="38" y1="17.75" x2="26.3" y2="17.75" width="0.3048" layer="1"/>
+<wire x1="26.3" y1="17.75" x2="23.5" y2="15.05" width="0.3048" layer="1"/>
+<wire x1="23.5" y1="15.05" x2="23.5" y2="12.65" width="0.3048" layer="1"/>
+<wire x1="23.5" y1="12.65" x2="22.25" y2="11.3" width="0.3048" layer="1"/>
+<wire x1="22.25" y1="11.3" x2="20.05" y2="11.3" width="0.3048" layer="1"/>
+<wire x1="20.05" y1="11.3" x2="18.45" y2="13.05" width="0.3048" layer="1"/>
+<wire x1="18.45" y1="13.05" x2="18.5" y2="20.8" width="0.3048" layer="1"/>
+<wire x1="18.5" y1="20.8" x2="17.05" y2="22.05" width="0.3048" layer="1"/>
+<via x="17.05" y="22.05" extent="1-16" drill="0.6" shape="octagon"/>
+<wire x1="17.05" y1="22.05" x2="14.61" y2="24.49" width="0.3048" layer="16"/>
+<wire x1="14.61" y1="24.49" x2="14.61" y2="41.97" width="0.3048" layer="16"/>
 </signal>
 <signal name="A0">

Commit message: Board revision big+5
Routing:
- net N$25: track 0.00 -> 88.0 mm, vias 0 -> 6
- net N$7: track 34.6 -> 82.0 mm, vias 2 -> 4
- net A0: track 8.57 -> 40.9 mm, vias 0 -> 2
- net A1: track 8.06 -> 36.4 mm, vias 0 -> 2
Changed lines of the file:
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@@
 <wire x1="49.85" y1="19.1" x2="48.25" y2="20.7" width="0.3048" layer="1"/>
 <wire x1="48.25" y1="20.7" x2="48.25" y2="21" width="0.3048" layer="1"/>
-<wire x1="19.69" y1="41.97" x2="52.2" y2="35.75" width="0" layer="19" extent="16-16"/>
+<via x="19.8" y="40.25" extent="1-16" drill="0.6" shape="octagon"/>
+<wire x1="19.8" y1="40.25" x2="19.75" y2="40.15" width="0.3048" layer="1"/>
+<wire x1="20.95" y1="41.15" x2="20.95" y2="43.7" width="0.3048" layer="1"/>
+<wire x1="20.95" y1="43.7" x2="23.75" y2="46.5" width="0.3048" layer="1"/>
+<wire x1="23.75" y1="46.5" x2="56.05" y2="46.5" width="0.3048" layer="1"/>
+<wire x1="56.05" y1="46.5" x2="57.65" y2="44.9" width="0.3048" layer="1"/>
+<via x="57.65" y="44.9" extent="1-16" drill="0.6" shape="octagon"/>
+<wire x1="57.65" y1="44.9" x2="57.65" y2="42.01" width="0.3048" layer="16"/>
+<wire x1="57.65" y1="42.01" x2="57.69" y2="41.97" width="0.3048" layer="16"/>
+<wire x1="19.69" y1="41.97" x2="19.69" y2="40.36" width="0.3048" layer="16"/>
+<wire x1="19.69" y1="40.36" x2="19.8" y2="40.25" width="0.3048" layer="16"/>
+<wire x1="20.95" y1="41.15" x2="20.7" y2="41.15" width="0.3048" layer="1"/>
+<wire x1="20.7" y1="41.15" x2="19.8" y2="40.25" width="0.3048" layer="1"/>
 </signal>
 <signal name="N$8">
@@
 <wire x1="43.5" y1="40.238" x2="45.675" y2="38.063" width="0.3048" layer="16"/>
 <wire x1="45.675" y1="38.063" x2="45.675" y2="33.08" width="0.3048" layer="16"/>
-<wire x1="57.69" y1="14.03" x2="45.675" y2="33.08" width="0" layer="19" extent="16-16"/>
+<wire x1="45.675" y1="33.08" x2="45.675" y2="32.375" width="0.3048" layer="16"/>
+<wire x1="45.675" y1="32.375" x2="49.75" y2="28.3" width="0.3048" layer="16"/>
+<wire x1="49.75" y1="28.3" x2="57.2" y2="28.3" width="0.3048" layer="16"/>
+<wire x1="57.2" y1="28.3" x2="57.45" y2="28.05" width="0.3048" layer="16"/>
+<via x="57.45" y="28.05" extent="1-16" drill="0.6" shape="octagon"/>
+<wire x1="57.45" y1="28.05" x2="57.45" y2="15.7" width="0.3048" layer="1"/>
+<wire x1="57.45" y1="15.7" x2="57.5" y2="15.65" width="0.3048" layer="1"/>
+<via x="57.5" y="15.65" extent="1-16" drill="0.6" shape="octagon"/>
+<wire x1="57.5" y1="15.65" x2="57.5" y2="14.22" width="0.3048" layer="16"/>
+<wire x1="57.5" y1="14.22" x2="57.69" y2="14.03" width="0.3048" layer="16"/>
 </signal>
 <signal name="N$10">
@@
 <contactref element="U2" pad="P$21"/>
 <contactref element="LED1" pad="6"/>
-<wire x1="41.865" y1="33.08" x2="65.31" y2="14.03" width="0" layer="19" extent="16-16"/>
+<wire x1="41.865" y1="33.08" x2="41.865" y2="31.415" width="0.3048" layer="16"/>
+<wire x1="41.865" y1="31.415" x2="41.45" y2="31" width="0.3048" layer="16"/>
+<wire x1="41.45" y1="31" x2="26.5" y2="31" width="0.3048" layer="16"/>
+<wire x1="26.5" y1="31" x2="20.75" y2="25.25" width="0.3048" layer="16"/>
+<via x="20.75" y="25.25" extent="1-16" drill="0.6" shape="octagon"/>
+<wire x1="20.75" y1="25.25" x2="20.75" y2="20.55" width="0.3048" layer="1"/>
+<wire x1="20.75" y1="20.55" x2="23.4" y2="17.8" width="0.3048" layer="1"/>
+<via x="23.4" y="17.8" extent="1-16" drill="0.6" shape="octagon"/>
+<wire x1="23.4" y1="17.8" x2="23.65" y2="17.5" width="0.3048" layer="16"/>
+<wire x1="23.65" y1="17.5" x2="26.05" y2="15.1" width="0.3048" layer="16"/>
+<wire x1="26.05" y1="15.1" x2="26.05" y2="12.2" width="0.3048" layer="16"/>
+<wire x1="26.05" y1="12.2" x2="28.6" y2="9.65" width="0.3048" layer="16"/>
+<via x="28.6" y="9.65" extent="1-16" drill="0.6" shape="octagon"/>
+<wire x1="28.6" y1="9.65" x2="38.55" y2="9.65" width="0.3048" layer="1"/>
+<wire x1="38.55" y1="9.65" x2="38.6" y2="9.6" width="0.3048" layer="1"/>
+<via x="38.6" y="9.6" extent="1-16" drill="0.6" shape="octagon"/>
+<wire x1="38.6" y1="9.6" x2="41.95" y2="9.6" width="0.3048" layer="16"/>
+<wire x1="41.95" y1="9.6" x2="43.35" y2="8.2" width="0.3048" layer="16"/>
+<wire x1="43.35" y1="8.2" x2="53.85" y2="8.2" width="0.3048" layer="16"/>
+<wire x1="53.85" y1="8.2" x2="53.95" y2="8.3" width="0.3048" layer="16"/>
+<via x="53.95" y="8.3" extent="1-16" drill="0.6" shape="octagon"/>
+<wire x1="53.95" y1="8.3" x2="56.55" y2="8.3" width="0.3048" layer="1"/>
+<wire x1="56.55" y1="8.3" x2="56.65" y2="8.4" width="0.3048" layer="1"/>
+<wire x1="56.65" y1="8.4" x2="57" y2="8.4" width="0.3048" layer="1"/>
+<wire x1="57" y1="8.4" x2="61.5" y2="13" width="0.3048" layer="1"/>
+<wire x1="61.5" y1="13" x2="61.5" y2="15.2" width="0.3048" layer="1"/>
+<wire x1="61.5" y1="15.2" x2="62.4" y2="16" width="0.3048" layer="1"/>
+<wire x1="62.4" y1="16" x2="64.65" y2="16" width="0.3048" layer="1"/>
+<wire x1="64.65" y1="16" x2="65.4" y2="15.9" width="0.3048" layer="1"/>
+<via x="65.4" y="15.9" extent="1-16" drill="0.6" shape="octagon"/>
+<wire x1="65.4" y1="15.9" x2="65.35" y2="14.07" width="0.3048" layer="16"/>
+<wire x1="65.35" y1="14.07" x2="65.31" y2="14.03" width="0.3048" layer="16"/>
 </signal>
 <signal name="N$26">
@@
 <wire x1="41" y1="40.238" x2="44.405" y2="36.833" width="0.3048" layer="16"/>
 <wire x1="44.405" y1="36.833" x2="44.405" y2="33.08" width="0.3048" layer="16"/>
-<wire x1="60.23" y1="14.03" x2="44.405" y2="33.08" width="0" layer="19" extent="16-16"/>
+<wire x1="44.405" y1="33.08" x2="44.405" y2="32.295" width="0.3048" layer="16"/>
+<wire x1="44.405" y1="32.295" x2="49.3" y2="27.4" width="0.3048" layer="16"/>
+<wire x1="49.3" y1="27.4" x2="55.65" y2="27.4" width="0.3048" layer="16"/>
+<wire x1="55.65" y1="27.4" x2="55.95" y2="27.1" width="0.3048" layer="16"/>
+<wire x1="55.95" y1="27.1" x2="60.05" y2="27.1" width="0.3048" layer="16"/>
+<wire x1="60.05" y1="27.1" x2="60.15" y2="27.4" width="0.3048" layer="16"/>
+<via x="60.15" y="27.4" extent="1-16" drill="0.6" shape="octagon"/>
+<wire x1="60.15" y1="27.4" x2="60.15" y2="15.75" width="0.3048" layer="1"/>
+<wire x1="60.15" y1="15.75" x2="60.2" y2="15.7" width="0.3048" layer="1"/>
+<via x="60.2" y="15.7" extent="1-16" drill="0.6" shape="octagon"/>
+<wire x1="60.2" y1="15.7" x2="60.2" y2="14.06" width="0.3048" layer="16"/>
+<wire x1="60.2" y1="14.06" x2="60.23" y2="14.03" width="0.3048" layer="16"/>
 </signal>
 <signal name="A2">

Commit message: Board revision big+6
Routing:
- net N$2: track 95.1 -> 90.1 mm
- net N$4: track 61.3 -> 58.3 mm
Changed lines of the file:
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@@
 <wire x1="17.15" y1="14.03" x2="17.15" y2="12.25" width="0.3048" layer="16"/>
 <via x="17.15" y="12.25" extent="1-16" drill="0.6" shape="octagon"/>
-<wire x1="17.15" y1="12.25" x2="21.4" y2="8" width="0.3048" layer="1"/>
-<wire x1="21.4" y1="8" x2="26.55" y2="8" width="0.3048" layer="1"/>
-<wire x1="26.55" y1="8" x2="28.25" y2="6.3" width="0.3048" layer="1"/>
-<wire x1="28.25" y1="6.3" x2="28.25" y2="2.65" width="0.3048" layer="1"/>
-<wire x1="28.25" y1="2.65" x2="28.65" y2="2.25" width="0.3048" layer="1"/>
-<wire x1="28.65" y1="2.25" x2="30.15" y2="2.25" width="0.3048" layer="1"/>
-<wire x1="30.15" y1="2.25" x2="33.9" y2="6" width="0.3048" layer="1"/>
+<wire x1="17.15" y1="12.25" x2="20.55" y2="9.05" width="0.3048" layer="1"/>
+<wire x1="20.55" y1="9.05" x2="25.7" y2="9.05" width="0.3048" layer="1"/>
+<wire x1="25.7" y1="9.05" x2="28.25" y2="6.3" width="0.3048" layer="1"/>
 <wire x1="33.9" y1="6" x2="34.15" y2="6" width="0.3048" layer="1"/>
 <via x="34.15" y="6" extent="1-16" drill="0.6" shape="octagon"/>
@@
 <wire x1="17.2" y1="19.7" x2="17.2" y2="14.08" width="0.3048" layer="16"/>
 <wire x1="17.2" y1="14.08" x2="17.15" y2="14.03" width="0.3048" layer="16"/>
+<wire x1="28.25" y1="6.3" x2="33.85" y2="6.3" width="0.3048" layer="1"/>
+<wire x1="33.85" y1="6.3" x2="34.15" y2="6" width="0.3048" layer="1"/>
 </signal>
 <signal name="N$3">
@@
 <wire x1="44.405" y1="14.03" x2="52.61" y2="14.03" width="0.3048" layer="16"/>
 <via x="44.405" y="14.03" extent="1-16" drill="0.6" shape="octagon"/>
-<wire x1="44.405" y1="14.03" x2="31.425" y2="1.05" width="0.3048" layer="1"/>
-<wire x1="31.425" y1="1.05" x2="27.9" y2="1.05" width="0.3048" layer="1"/>
-<wire x1="27.9" y1="1.05" x2="26.75" y2="2.2" width="0.3048" layer="1"/>
-<wire x1="26.75" y1="2.2" x2="26.75" y2="5.8" width="0.3048" layer="1"/>
-<wire x1="26.75" y1="5.8" x2="25.8" y2="6.75" width="0.3048" layer="1"/>
-<wire x1="25.8" y1="6.75" x2="19.35" y2="6.75" width="0.3048" layer="1"/>
-<wire x1="19.35" y1="6.75" x2="14.55" y2="11.55" width="0.3048" layer="1"/>
+<wire x1="27.65" y1="5.8" x2="25.05" y2="8.05" width="0.3048" layer="1"/>
+<wire x1="25.05" y1="8.05" x2="18.6" y2="8.05" width="0.3048" layer="1"/>
+<wire x1="18.6" y1="8.05" x2="14.55" y2="11.55" width="0.3048" layer="1"/>
 <wire x1="14.55" y1="11.55" x2="14.55" y2="12.2" width="0.3048" layer="1"/>
 <via x="14.55" y="12.2" extent="1-16" drill="0.6" shape="octagon"/>
 <wire x1="14.55" y1="12.2" x2="14.61" y2="12.26" width="0.3048" layer="16"/>
 <wire x1="14.61" y1="12.26" x2="14.61" y2="14.03" width="0.3048" layer="16"/>
+<wire x1="35" y1="4.45" x2="39" y2="8.45" width="0.3048" layer="1"/>
+<wire x1="39" y1="8.45" x2="42.55" y2="8.45" width="0.3048" layer="1"/>
+<wire x1="42.55" y1="8.45" x2="44.4" y2="10.3" width="0.3048" layer="1"/>
+<wire x1="44.4" y1="10.3" x2="44.4" y2="14.025" width="0.3048" layer="1"/>
+<wire x1="44.4" y1="14.025" x2="44.405" y2="14.03" width="0.3048" layer="1"/>
+<wire x1="27.65" y1="5.8" x2="29" y2="4.45" width="0.3048" layer="1"/>
+<wire x1="29" y1="4.45" x2="35" y2="4.45" width="0.3048" layer="1"/>
 </signal>
 <signal name="N$6">
@@
 <contactref element="SV1" pad="9"/>
 <contactref element="SV2" pad="2"/>
-<polygon width="0.3048" layer="1">
+<polygon width="0.3048" layer="1" isolate="0.6096">
 <vertex x="0" y="55.88"/>
 <vertex x="0" y="0"/>
@@
 <vertex x="86.36" y="55.88"/>
 </polygon>
-<polygon width="0.3048" layer="16">
+<polygon width="0.3048" layer="16" isolate="0.6096">
 <vertex x="0" y="55.88"/>
 <vertex x="0" y="0"/>
@@
 <vertex x="86.36" y="55.88"/>
 </polygon>
+<via x="52.6" y="22.9" extent="1-16" drill="0.6" shape="octagon"/>
+<via x="61.6" y="35.45" extent="1-16" drill="0.6" shape="octagon"/>
+<wire x1="33.45270625" y1="53.77" x2="38.53270625" y2="51.23" width="0" layer="19" extent="1-1"/>
 </signal>
 <signal name="N$19">
