File: eagle/MatrixPi.brd (EAGLE design)
At the start: 85 x 56 mm, 17 parts, among them U2 28-SOIC

Commit message: brd
Routing:
- net N$4: track 58.3 -> 59.0 mm

Commit message: updated board
Routing:
- net N$6: track 80.3 -> 68.7 mm
- net N$41: track 87.2 -> 76.6 mm
- net N$39: track 102.7 -> 93.1 mm
- net N$2: track 90.0 -> 83.2 mm
- net N$3: track 78.4 -> 72.1 mm
- net N$22: track 22.8 -> 24.9 mm
- net N$1: track 70.7 -> 72.3 mm
- net SDA: track 69.3 -> 67.7 mm
- net N$7: track 82.3 -> 80.9 mm
- net A0: track 40.9 -> 41.7 mm
